File: kicad/kicad.kicad_pcb (KiCad board)
At the start: 2 copper layers, 323.8 x 104.8 mm, 138 parts, among them J1 USB_C_Receptacle_USB2.0_14P, J2 Conn_01x02_Pin, SW1 ROT_SKYLOONG_HS, SW2 ROT_SKYLOONG_HS, SW3 ROT_SKYLOONG_HS, SW4 ROT_SKYLOONG_HS, U1 RP2040, U2 NCP1117-3.3_SOT223, U3 W25Q128JVS, X1 ABM8-272-T3

Commit message: rehaul
Parts:
- added 2uStabilizer1: MX_stab, PCM_marbastlib-mx:STAB_MX_2u, B.Cu at (218.8, 114.4)
- added Spacebar1: MX_SW_HS, PCM_marbastlib-mx:SW_MX_HS_CPG151101S11_1u, B.Cu at (218.8, 114.4)
- moved D23 163.8 mm to (190.5, 16.7)
- moved MX56 163.8 mm to (190.5, 54.8)
- moved MX69 163.8 mm to (190.5, 73.9)
- moved MX70 163.8 mm to (190.5, 92.9)
- moved SW1 161.7 mm to (189.8, 29.3)
- moved MX55 158.1 mm to (141.4, 167.5)
- moved D21 117.1 mm to (421.5, 109.5)
- moved D25 117.1 mm to (431.0, 38.1)
- moved D26 117.1 mm to (450.0, 38.1)
- moved D29 117.1 mm to (421.5, 85.7)
- moved MX14 117.1 mm to (431.0, 57.1)
- moved MX28 117.1 mm to (431.0, 76.2)
- moved MX42 117.1 mm to (431.0, 95.2)
- moved MX54 117.1 mm to (431.0, 114.3)
- moved MX71 117.1 mm to (450.0, 57.1)
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Routing:
- net Row 5: track 249.8 -> 322.6 mm
- net Net-(D19-A2): track 30.3 -> 93.8 mm
- net Column 8: track 89.7 -> 148.8 mm
Other:
- board size 323.8 x 104.8 mm -> 423.1 x 104.8 mm
- rule pad_to_mask_clearance: 0 -> 0.051
