File: pcb_and_schematic/SKBD/_autosave-SKBD.kicad_sch (KiCad schematic)
At the start: 150 parts, among them J2 USB_C_Receptacle_USB2.0_14P, SW1 ROT_SKYLOONG_HS, SW10 ROT_SKYLOONG_HS, SW11 ROT_SKYLOONG_HS, SW12 Push_Button, SW2 ROT_SKYLOONG_HS, SW3 ROT_SKYLOONG_HS, SW4 ROT_SKYLOONG_HS, SW5 ROT_SKYLOONG_HS, SW6 ROT_SKYLOONG_HS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

Commit message: rehaul
Connections:
- net at MX11.1, MX23.1, MX35.1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: now also MX10.1, MX12.1, MX22.1, MX24.1, MX34.1, MX36.1, MX46.1, MX48.1, MX57.1, MX59.1
- net at MX19.1, MX31.1, MX43.1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: now also MX20.1, MX21.1, MX32.1, MX33.1, MX44.1, MX45.1, MX55.1, MX56.1, MX8.1, MX9.1
Changed lines of the file:
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@@
 	)
 	(junction
+		(at 307.34 63.5)
+		(diameter 0)
+		(color 0 0 0 0)
+	)
+	(junction
 		(at 463.55 119.38)
 		(diameter 0)
@@
 	)
 	(junction
+		(at 256.54 63.5)
+		(diameter 0)
+		(color 0 0 0 0)
+	)
+	(junction
 		(at 483.87 99.06)
 		(diameter 0)
@@
 	(wire
 		(pts
+			(xy 307.34 63.5) (xy 325.12 63.5)
+		)
+		(stroke
+			(width 0)
+			(type default)
+		)
+	)
+	(wire
+		(pts
 			(xy 345.44 200.66) (xy 345.44 161.29)
 		)
@@
 	(wire
 		(pts
+			(xy 243.84 63.5) (xy 256.54 63.5)
+		)
+		(stroke
+			(width 0)
+			(type default)
+		)
+	)
+	(wire
+		(pts
 			(xy 91.44 102.87) (xy 91.44 109.22)
 		)
@@
 	(wire
 		(pts
+			(xy 256.54 63.5) (xy 274.32 63.5)
+		)
+		(stroke
+			(width 0)
+			(type default)
+		)
+	)
+	(wire
+		(pts
 			(xy 359.41 119.38) (xy 358.14 119.38)
 		)
@@
 		)
 		(stroke
+			(width 0)
+			(type default)
+		)
+	)
+	(wire
+		(pts
+			(xy 294.64 63.5) (xy 307.34 63.5)
+		)
+		(stroke
