File: pcb_and_schematic/SKBD/SKBD.kicad_pcb (KiCad board)
At the start: 2 copper layers, 323.8 x 95.2 mm, 150 parts, among them J2 USB_C_Receptacle_USB2.0_14P, SW1 ROT_SKYLOONG_HS, SW10 ROT_SKYLOONG_HS, SW11 ROT_SKYLOONG_HS, SW12 Slide_Switch_SPDT_P3mm_10x5x1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, SW2 ROT_SKYLOONG_HS, SW3 ROT_SKYLOONG_HS, SW4 ROT_SKYLOONG_HS, SW5 ROT_SKYLOONG_HS, SW6 ROT_SKYLOONG_HS, SW7 ROT_SKYLOONG_HS, SW8 ROT_SKYLOONG_HS, SW9 ROT_SKYLOONG_HS, U2 NCP1117-3.3_SOT223, U3 W25Q128JVS, U4 RP2040, Y1 ABM8-272-T3

Commit message: wiring
Parts:
- moved U3 0.38 mm to (107.0, 59.3)
Routing:
- net Net-(D12-K3): track 0.00 -> 321.5 mm
- net Net-(D10-K1): track 0.00 -> 320.7 mm
- net Net-(D12-K2): track 0.00 -> 320.6 mm
- net Net-(D13-K1): track 0.00 -> 307.1 mm
- net Net-(D13-K2): track 0.00 -> 306.1 mm
- net Net-(MX21-Pad1): track 0.00 -> 76.2 mm
- net Net-(D9-A1): track 0.00 -> 28.5 mm
- net Net-(D33-A1): track 0.00 -> 25.9 mm
- net Net-(D32-A1): track 0.00 -> 25.9 mm
- net Net-(D17-A1): track 0.00 -> 25.9 mm
- net Net-(D16-A1): track 0.00 -> 25.9 mm
- net Net-(D11-A1): track 0.00 -> 25.9 mm
- net Net-(D10-A1): track 0.00 -> 25.9 mm
- net Net-(D8-A1): track 0.00 -> 25.9 mm
- net Net-(D14-A1): track 0.00 -> 25.9 mm
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
Commit message: wiring update
Parts:
- SW12: value Slide_Switch_SPDT_P3mm_10x5x10mm -> Push_Button; footprint PCM_SL_Devices:Slide_Switch_SPDT_P3mm_10x5x10mm -> PCM_marbastlib-various:SW_SPST_SKQG_WithStem; moved to B.Cu
- moved SW12 266.4 mm to (128.6, 57.1), turned to 180 degrees
- moved R7 259.6 mm to (83.2, 22.4)
- moved R6 255.9 mm to (81.7, 24.7)
- moved C3 251.9 mm to (90.5, 34.2)
- moved C5 245.1 mm to (109.4, 56.1), turned to 0 degrees
- moved R1 233.3 mm to (109.4, 61.1), turned to 0 degrees
- moved R2 233.3 mm to (109.4, 63.1)
- moved U3 2.06 mm to (105.0, 59.7)
- moved U2 0.63 mm to (90.5, 40.2)
- moved J2 0.09 mm to (90.5, 21.9)
Connections:
- SW12 pad 1: /~{USB_BOOT} -> GND
- SW12 pad 2: GND -> /~{USB_BOOT}
Routing:
- net Net-(D19-K1): track 0.00 -> 310.2 mm
- net Net-(D19-K2): track 0.00 -> 309.3 mm
- net Net-(D19-K3): track 0.00 -> 306.1 mm
- net Net-(D25-K2): track 0.00 -> 302.7 mm
- net Net-(D25-K1): track 0.00 -> 302.1 mm, vias 0 -> 4
- net Net-(D25-K3): track 0.00 -> 299.0 mm
- net Net-(D28-A3): track 0.00 -> 39.5 mm
- net Net-(D29-A3): track 0.00 -> 29.5 mm
- net Net-(D26-A3): track 0.00 -> 29.5 mm
- net Net-(D27-A3): track 0.00 -> 29.5 mm
- net Net-(D23-A1): track 0.00 -> 25.9 mm
- net Net-(D34-A1): track 0.00 -> 25.9 mm
- net Net-(D22-A1): track 0.00 -> 25.9 mm
- net Net-(D20-A1): track 0.00 -> 25.9 mm
- net Net-(D21-A1): track 0.00 -> 25.9 mm
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
Commit message: wiring change
Parts:
- moved R5 238.5 mm to (93.2, 37.6), turned to 0 degrees
- moved R4 237.8 mm to (93.2, 36.6), turned to 0 degrees
- moved U2 22.6 mm to (105.8, 23.6), turned to 0 degrees
- moved SW12 19.0 mm to (128.6, 38.1)
- moved C5 18.4 mm to (109.4, 37.7)
- moved R1 18.4 mm to (109.4, 42.7)
- moved R2 18.4 mm to (109.4, 44.7)
- moved U3 18.4 mm to (105.0, 41.2)
- moved U4 18.4 mm to (90.5, 42.4)
- moved C3 13.4 mm to (98.6, 23.6), turned to -90 degrees
Connections:
- net Net-(U2-VI) renamed VBUS
Routing:
- net Net-(D1-K3): track 305.1 -> 323.3 mm
- net VBUS: track 0.00 -> 16.4 mm
- net Net-(D1-K2): track 307.0 -> 321.5 mm
- net Net-(D1-K1): track 307.9 -> 322.2 mm
- net /USB_D-: track 0.00 -> 8.31 mm
- net /USB_D+: track 0.00 -> 5.44 mm
- net Net-(D9-A1): track 28.5 -> 25.9 mm
- net Net-(D3-A1): track 25.9 -> 27.7 mm
- net /~{USB_BOOT}: track 22.6 -> 23.9 mm
- net Net-(MX16-Pad1): track 238.7 -> 238.1 mm
- added copper zone on B.Cu, net VBUS

Commit message: wiring change
Parts:
- moved C17 283.0 mm to (116.9, 23.6), turned to -90 degrees
- moved C4 277.3 mm to (112.1, 23.6), turned to -90 degrees
- moved C11 246.3 mm to (97.7, 44.1), turned to 0 degrees
- moved C15 246.0 mm to (96.7, 45.1), turned to 0 degrees
- moved C16 245.8 mm to (95.8, 46.1), turned to 0 degrees
- moved C6 244.8 mm to (94.8, 39.4), turned to 0 degrees
- moved C10 243.8 mm to (89.4, 36.0)
- moved C14 243.2 mm to (88.4, 37.2)
- moved C8 243.2 mm to (93.4, 37.8), turned to 0 degrees
- moved C12 242.0 mm to (85.6, 38.3)
- moved C13 238.4 mm to (85.6, 39.3)
- moved C7 234.6 mm to (83.3, 43.7)
- moved C9 233.1 mm to (84.4, 44.7)
- moved C2 229.2 mm to (80.9, 43.2), turned to 90 degrees
- moved C1 224.9 mm to (78.1, 44.6), turned to 0 degrees
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Connections:
- D1 pad 4: Net-(D1-K3) -> Row 1
- D2 pad 4: Net-(D1-K3) -> Row 1
- D2 pad 5: Net-(D1-K3) -> Row 1
- D2 pad 6: Net-(D1-K3) -> Row 1
- D3 pad 4: Net-(D1-K3) -> Row 1
- D3 pad 5: Net-(D1-K3) -> Row 1
- D3 pad 6: Net-(D1-K3) -> Row 1
- D4 pad 4: Net-(D1-K3) -> Row 1
- D4 pad 5: Net-(D1-K3) -> Row 1
- D4 pad 6: Net-(D1-K3) -> Row 1
- D5 pad 4: Net-(D1-K3) -> Row 1
- D5 pad 5: Net-(D1-K3) -> Row 1
- D5 pad 6: Net-(D1-K3) -> Row 1
- D6 pad 6: Net-(D1-K3) -> Row 1
- U4 pad 11: Col. 9 -> unconnected-(U4-GPIO8-Pad11)
- U4 pad 12: Col. 10 -> unconnected-(U4-GPIO9-Pad12)
- U4 pad 13: Col. 11 -> unconnected-(U4-GPIO10-Pad13)
- U4 pad 14: Col. 12 -> unconnected-(U4-GPIO11-Pad14)
- U4 pad 15: Col. 13 -> unconnected-(U4-GPIO12-Pad15)
- U4 pad 16: Col. 14 -> unconnected-(U4-GPIO13-Pad16)
- U4 pad 17: Row 1 -> unconnected-(U4-GPIO14-Pad17)
- U4 pad 18: Row 2 -> unconnected-(U4-GPIO15-Pad18)
- U4 pad 2: Col. 1 -> Row 1
- U4 pad 27: Row 3 -> unconnected-(U4-GPIO16-Pad27)
- U4 pad 28: Row 4 -> unconnected-(U4-GPIO17-Pad28)
- U4 pad 29: Row 5 -> unconnected-(U4-GPIO18-Pad29)
- U4 pad 3: Col. 2 -> unconnected-(U4-GPIO1-Pad3)
- U4 pad 30: Rot. Enc A1 -> unconnected-(U4-GPIO19-Pad30)
- U4 pad 31: Rot. Enc B1 -> unconnected-(U4-GPIO20-Pad31)
- U4 pad 32: Rot. Enc A2 -> unconnected-(U4-GPIO21-Pad32)
- U4 pad 34: Rot. Enc B2 -> unconnected-(U4-GPIO22-Pad34)
- U4 pad 35: Rot. Enc A3 -> unconnected-(U4-GPIO23-Pad35)
- U4 pad 36: Rot. Enc B3 -> unconnected-(U4-GPIO24-Pad36)
- U4 pad 37: Rot. Enc A4 -> unconnected-(U4-GPIO25-Pad37)
- U4 pad 38: Rot. Enc B4 -> unconnected-(U4-GPIO26_ADC0-Pad38)
- U4 pad 39: Rot. Enc A5 -> unconnected-(U4-GPIO27_ADC1-Pad39)
- U4 pad 4: Col. 3 -> unconnected-(U4-GPIO2-Pad4)
- U4 pad 40: Rot. Enc B5 -> unconnected-(U4-GPIO28_ADC2-Pad40)
- U4 pad 41: Col. 15 -> unconnected-(U4-GPIO29_ADC3-Pad41)
- U4 pad 5: Col. 4 -> unconnected-(U4-GPIO3-Pad5)
- U4 pad 6: Col. 5 -> unconnected-(U4-GPIO4-Pad6)
- U4 pad 7: Col. 6 -> unconnected-(U4-GPIO5-Pad7)
- U4 pad 8: Col. 7 -> unconnected-(U4-GPIO6-Pad8)
- U4 pad 9: Col. 8 -> unconnected-(U4-GPIO7-Pad9)
Routing:
- net Row 1: track 0.00 -> 330.9 mm, vias 0 -> 2
- net Net-(D1-K3): track 323.3 -> 0.00 mm
- net GND: track 0.00 -> 52.2 mm, vias 0 -> 23
- net +3V3: track 2.03 -> 31.8 mm, vias 0 -> 2
- net Net-(D10-K1): track 322.1 -> 305.3 mm
- net /XIN: track 0.00 -> 16.8 mm
- net Net-(D12-K2): track 320.6 -> 306.3 mm
- net Net-(D12-K3): track 321.6 -> 307.3 mm
- net /USB_D+: track 5.44 -> 18.2 mm
- net +1V1: track 0.00 -> 7.53 mm
- net /USB_D-: track 8.31 -> 15.7 mm
- net Net-(C2-Pad1): track 0.00 -> 6.83 mm
- net Net-(MX15-Pad1): track 76.2 -> 82.2 mm
- net Net-(U4-USB_DP): track 0.00 -> 4.23 mm
- net Net-(U4-USB_DM): track 0.00 -> 3.40 mm
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- added copper zone on B.Cu, net +3V3
- added copper zone on F.Cu, net GND

Commit message: revert to old desing
Parts:
- removed J2: USB_C_Receptacle_USB2.0_14P, Connector_USB:USB_C_Receptacle_JAE_DX07S016JA1R1500
- added D36: PRTR5V0U2X, Package_TO_SOT_SMD:SOT-143, B.Cu at (52.4, 47.5)
- added USB1: HRO-TYPE-C-31-M-12, Type-C:HRO-TYPE-C-31-M-12-Assembly, B.Cu at (52.4, 32.7)
- C1, C10, C11, C12, C13, C14, C15, C16, C2, C5, C6, C7, C8, C9: footprint Capacitor_SMD:C_0402_1005Metric -> Capacitor_SMD:C_0805_2012Metric
- R1, R2, R3, R4, R5: footprint Resistor_SMD:R_0402_1005Metric -> Resistor_SMD:R_0805_2012Metric
- R6, R7: footprint Resistor_SMD:R_01005_0402Metric -> Resistor_SMD:R_0805_2012Metric
- S2: moved to F.Cu
- moved C17 178.9 mm to (-60.8, 44.1), turned to 180 degrees
- moved C5 177.9 mm to (-56.7, 99.7), turned to 180 degrees
- moved C4 173.8 mm to (-60.8, 41.1), turned to 180 degrees
- moved R1 169.3 mm to (-53.9, 87.5), turned to 180 degrees
- moved R2 169.3 mm to (-53.9, 89.5)
- moved C15 168.3 mm to (-62.5, 99.7), turned to 180 degrees
- moved C16 167.7 mm to (-62.5, 101.7), turned to 180 degrees
- moved C11 167.5 mm to (-59.6, 101.7), turned to 180 degrees
- moved C6 163.8 mm to (-56.7, 101.7), turned to 180 degrees
- moved C8 163.6 mm to (-59.6, 95.8), turned to 180 degrees
- moved C14 162.6 mm to (-62.5, 97.8)
- moved C10 162.1 mm to (-59.6, 99.7)
- moved C12 159.2 mm to (-59.6, 103.7)
- moved C13 158.5 mm to (-62.5, 95.8)
- moved C9 153.5 mm to (-59.6, 97.8)
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Connections:
- D1 pad 5: Net-(D1-K2) -> Row 2
- D1 pad 6: Net-(D1-K1) -> Row 3
- D10 pad 4: Net-(D10-K1) -> Row 6
- D10 pad 5: Net-(D10-K1) -> Row 5
- D10 pad 6: Net-(D10-K1) -> Row 4
- D11 pad 4: Net-(D10-K1) -> Row 6
- D11 pad 5: Net-(D10-K1) -> Row 5
- D11 pad 6: Net-(D10-K1) -> Row 4
- D12 pad 4: Net-(D12-K3) -> Row 6
- D12 pad 5: Net-(D12-K2) -> Row 5
- D12 pad 6: Net-(D10-K1) -> Row 4
- D13 pad 4: Net-(D13-K3) -> Row 7
- D13 pad 5: Net-(D13-K2) -> Row 8
- D13 pad 6: Net-(D13-K1) -> Row 9
- D14 pad 4: Net-(D13-K3) -> Row 9
- D14 pad 5: Net-(D13-K3) -> Row 8
- D14 pad 6: Net-(D13-K3) -> Row 7
- D15 pad 4: Net-(D13-K3) -> Row 9
- D15 pad 5: Net-(D13-K3) -> Row 8
- D15 pad 6: Net-(D13-K3) -> Row 7
- D16 pad 4: Net-(D13-K3) -> Row 9
- D16 pad 5: Net-(D13-K3) -> Row 8
- D16 pad 6: Net-(D13-K3) -> Row 7
- D17 pad 4: Net-(D13-K3) -> Row 9
- D17 pad 5: Net-(D13-K3) -> Row 8
- D17 pad 6: Net-(D13-K3) -> Row 7
- D18 pad 4: Net-(D13-K1) -> Row 9
- D18 pad 5: Net-(D13-K2) -> Row 8
- D18 pad 6: Net-(D13-K3) -> Row 7
- D19 pad 4: Net-(D19-K3) -> Row 10
- D19 pad 5: Net-(D19-K2) -> Row 11
- D19 pad 6: Net-(D19-K1) -> Row 12
- D2 pad 4: Row 1 -> Row 3
- D2 pad 5: Row 1 -> Row 2
- D20 pad 4: Net-(D19-K3) -> Row 12
- D20 pad 5: Net-(D19-K3) -> Row 11
- D20 pad 6: Net-(D19-K3) -> Row 10
- D21 pad 4: Net-(D19-K3) -> Row 12
- D21 pad 5: Net-(D19-K3) -> Row 11
- D21 pad 6: Net-(D19-K3) -> Row 10
- D22 pad 4: Net-(D19-K3) -> Row 12
- D22 pad 5: Net-(D19-K3) -> Row 11
- D22 pad 6: Net-(D19-K3) -> Row 10
- D23 pad 4: Net-(D19-K3) -> Row 12
- D23 pad 5: Net-(D19-K3) -> Row 11
- D23 pad 6: Net-(D19-K3) -> Row 10
- D24 pad 4: Net-(D19-K1) -> Row 12
- D24 pad 5: Net-(D19-K2) -> Row 11
- D24 pad 6: Net-(D19-K3) -> Row 10
- D25 pad 4: Net-(D25-K3) -> Row 14
- D25 pad 5: Net-(D25-K2) -> Row 15
- D25 pad 6: Net-(D25-K1) -> Row 16
- D26 pad 4: Net-(D25-K3) -> Row 14
- D26 pad 5: Net-(D25-K3) -> Row 15
- D26 pad 6: Net-(D25-K3) -> Row 16
- D27 pad 4: Net-(D25-K3) -> Row 14
- D27 pad 5: Net-(D25-K3) -> Row 15
- D27 pad 6: Net-(D25-K3) -> Row 16
- D28 pad 4: Net-(D25-K3) -> Row 14
- D28 pad 5: Net-(D25-K3) -> Row 15
- D28 pad 6: Net-(D25-K3) -> Row 16
- D29 pad 4: Net-(D25-K3) -> Row 14
- D29 pad 5: Net-(D25-K3) -> Row 15
- D29 pad 6: Net-(D25-K3) -> Row 16
- D3 pad 4: Row 1 -> Row 3
- D3 pad 5: Row 1 -> Row 2
- D30 pad 4: Net-(D25-K3) -> Row 14
- D30 pad 5: Net-(D25-K2) -> Row 15
- D30 pad 6: Net-(D25-K1) -> Row 16
- D31 pad 4: Net-(D1-K2) -> Row 3
- D31 pad 5: Net-(D1-K2) -> Row 2
- D31 pad 6: Net-(D1-K2) -> Row 1
- D32 pad 4: Net-(D12-K2) -> Row 6
- D32 pad 5: Net-(D12-K2) -> Row 5
- D32 pad 6: Net-(D12-K2) -> Row 4
- D33 pad 4: Net-(D13-K2) -> Row 9
- D33 pad 5: Net-(D13-K2) -> Row 8
- D33 pad 6: Net-(D13-K2) -> Row 7
- D34 pad 4: Net-(D19-K2) -> Row 12
- D34 pad 5: Net-(D19-K2) -> Row 11
- D34 pad 6: Net-(D19-K2) -> Row 10
- D35 pad 4: Net-(D25-K3) -> Row 14
- D35 pad 5: Net-(D25-K1) -> Row 16
- D35 pad 6: Net-(D25-K2) -> Row 15
- D4 pad 4: Row 1 -> Row 3
- D4 pad 5: Row 1 -> Row 2
- D5 pad 4: Row 1 -> Row 3
- D5 pad 5: Row 1 -> Row 2
- D6 pad 4: Net-(D1-K1) -> Row 3
- D6 pad 5: Net-(D1-K2) -> Row 2
- D7 pad 4: Net-(D10-K1) -> Row 4
- D7 pad 5: Net-(D12-K2) -> Row 5
- D7 pad 6: Net-(D12-K3) -> Row 6
- D8 pad 4: Net-(D10-K1) -> Row 6
- D8 pad 5: Net-(D10-K1) -> Row 5
- D8 pad 6: Net-(D10-K1) -> Row 4
- D9 pad 4: Net-(D10-K1) -> Row 6
- D9 pad 5: Net-(D10-K1) -> Row 5
- D9 pad 6: Net-(D10-K1) -> Row 4
- MX1 pad 1: Net-(MX1-Pad1) -> Col 2
- MX10 pad 1: Net-(MX10-Pad1) -> Col 7
- MX11 pad 1: Net-(MX11-Pad1) -> Col 7
- MX12 pad 1: Net-(MX12-Pad1) -> Col 7
- MX13 pad 1: Net-(MX1-Pad1) -> Col 2
- MX14 pad 1: Net-(MX14-Pad1) -> Col 2
- MX15 pad 1: Net-(MX15-Pad1) -> Col 2
- MX16 pad 1: Net-(MX16-Pad1) -> Col 3
- MX17 pad 1: Net-(MX17-Pad1) -> Col 3
- MX18 pad 1: Net-(MX18-Pad1) -> Col 3
- MX19 pad 1: Net-(MX19-Pad1) -> Col 6
- MX2 pad 1: Net-(MX14-Pad1) -> Col 2
- MX20 pad 1: Net-(MX20-Pad1) -> Col 6
- MX21 pad 1: Net-(MX21-Pad1) -> Col 6
- MX22 pad 1: Net-(MX10-Pad1) -> Col 7
- MX23 pad 1: Net-(MX11-Pad1) -> Col 7
- MX24 pad 1: Net-(MX12-Pad1) -> Col 7
- MX25 pad 1: Net-(MX1-Pad1) -> Col 2
- MX26 pad 1: Net-(MX14-Pad1) -> Col 2
- MX27 pad 1: Net-(MX15-Pad1) -> Col 2
- MX28 pad 1: Net-(MX16-Pad1) -> Col 3
- MX29 pad 1: Net-(MX17-Pad1) -> Col 3
- MX3 pad 1: Net-(MX15-Pad1) -> Col 2
- MX30 pad 1: Net-(MX18-Pad1) -> Col 3
- MX31 pad 1: Net-(MX19-Pad1) -> Col 6
- MX32 pad 1: Net-(MX20-Pad1) -> Col 6
- MX33 pad 1: Net-(MX21-Pad1) -> Col 6
- MX34 pad 1: Net-(MX10-Pad1) -> Col 7
- MX35 pad 1: Net-(MX11-Pad1) -> Col 7
- MX36 pad 1: Net-(MX12-Pad1) -> Col 7
- MX37 pad 1: Net-(MX1-Pad1) -> Col 2
- MX38 pad 1: Net-(MX14-Pad1) -> Col 2
- MX39 pad 1: Net-(MX15-Pad1) -> Col 2
- MX4 pad 1: Net-(MX16-Pad1) -> Col 3
- MX40 pad 1: Net-(MX16-Pad1) -> Col 3
- MX41 pad 1: Net-(MX17-Pad1) -> Col 3
- MX42 pad 1: Net-(MX18-Pad1) -> Col 3
- MX43 pad 1: Net-(MX19-Pad1) -> Col 6
- MX44 pad 1: Net-(MX20-Pad1) -> Col 6
- MX45 pad 1: Net-(MX21-Pad1) -> Col 6
- MX46 pad 1: Net-(MX10-Pad1) -> Col 7
- MX47 pad 1: Net-(MX11-Pad1) -> Col 7
- MX48 pad 1: Net-(MX12-Pad1) -> Col 7
- MX49 pad 1: Net-(MX1-Pad1) -> Col 2
- MX5 pad 1: Net-(MX17-Pad1) -> Col 3
- MX50 pad 1: Net-(MX14-Pad1) -> Col 2
- MX51 pad 1: Net-(MX15-Pad1) -> Col 2
- MX52 pad 1: Net-(MX16-Pad1) -> Col 3
- MX53 pad 1: Net-(MX17-Pad1) -> Col 3
- MX54 pad 1: Net-(MX18-Pad1) -> Col 3
- MX55 pad 1: Net-(MX20-Pad1) -> Col 6
- MX56 pad 1: Net-(MX21-Pad1) -> Col 6
- MX57 pad 1: Net-(MX10-Pad1) -> Col 7
- MX58 pad 1: Net-(MX11-Pad1) -> Col 7
- MX59 pad 1: Net-(MX12-Pad1) -> Col 7
- MX6 pad 1: Net-(MX18-Pad1) -> Col 3
- MX60 pad 1: Net-(MX19-Pad1) -> Col 6
- MX61 pad 1: Net-(MX18-Pad1) -> Col 4
- MX62 pad 1: Net-(MX17-Pad1) -> Col 4
- MX63 pad 1: Net-(MX16-Pad1) -> Col 4
- MX64 pad 1: Net-(MX18-Pad1) -> Col 4
- MX65 pad 1: Net-(MX17-Pad1) -> Col 4
- MX66 pad 1: Net-(MX16-Pad1) -> Col 4
- MX67 pad 1: Net-(MX18-Pad1) -> Col 4
- MX68 pad 1: Net-(MX17-Pad1) -> Col 4
- MX69 pad 1: Net-(MX16-Pad1) -> Col 4
- MX7 pad 1: Net-(MX19-Pad1) -> Col 6
- MX70 pad 1: Net-(MX18-Pad1) -> Col 4
- MX71 pad 1: Net-(MX17-Pad1) -> Col 4
- MX72 pad 1: Net-(MX16-Pad1) -> Col 4
- MX8 pad 1: Net-(MX20-Pad1) -> Col 6
- MX9 pad 1: Net-(MX21-Pad1) -> Col 6
- SW1 pad C: Net-(SW1-PadC) -> Col 1
- SW10 pad C: Net-(SW10-PadC) -> Col 8
- SW11 pad C: unconnected-(SW11-PadC) -> Col 4
- SW2 pad C: Net-(SW10-PadC) -> Col 8
- SW3 pad C: Net-(SW1-PadC) -> Col 1
- SW4 pad C: Net-(SW10-PadC) -> Col 8
- SW5 pad C: Net-(SW1-PadC) -> Col 1
- SW6 pad C: Net-(SW10-PadC) -> Col 8
- SW7 pad C: Net-(SW1-PadC) -> Col 1
- SW8 pad C: Net-(SW10-PadC) -> Col 8
- SW9 pad C: Net-(SW1-PadC) -> Col 1
- U4 pad 11: unconnected-(U4-GPIO8-Pad11) -> Row 9
- U4 pad 12: unconnected-(U4-GPIO9-Pad12) -> Row 10
- U4 pad 13: unconnected-(U4-GPIO10-Pad13) -> Row 11
- U4 pad 14: unconnected-(U4-GPIO11-Pad14) -> Row 12
- U4 pad 15: unconnected-(U4-GPIO12-Pad15) -> Row 14
- U4 pad 16: unconnected-(U4-GPIO13-Pad16) -> Row 15
- U4 pad 17: unconnected-(U4-GPIO14-Pad17) -> Row 16
- U4 pad 18: unconnected-(U4-GPIO15-Pad18) -> Col 1
- U4 pad 27: unconnected-(U4-GPIO16-Pad27) -> Col 2
- U4 pad 28: unconnected-(U4-GPIO17-Pad28) -> Col 3
- U4 pad 29: unconnected-(U4-GPIO18-Pad29) -> Col 4
- U4 pad 3: unconnected-(U4-GPIO1-Pad3) -> Row 2
- U4 pad 30: unconnected-(U4-GPIO19-Pad30) -> Col 6
- U4 pad 31: unconnected-(U4-GPIO20-Pad31) -> Col 7
- U4 pad 32: unconnected-(U4-GPIO21-Pad32) -> Col 8
- U4 pad 4: unconnected-(U4-GPIO2-Pad4) -> Row 3
- U4 pad 5: unconnected-(U4-GPIO3-Pad5) -> Row 4
- U4 pad 6: unconnected-(U4-GPIO4-Pad6) -> Row 5
- U4 pad 7: unconnected-(U4-GPIO5-Pad7) -> Row 6
- U4 pad 8: unconnected-(U4-GPIO6-Pad8) -> Row 7
- U4 pad 9: unconnected-(U4-GPIO7-Pad9) -> Row 8
Routing:
- net Net-(D1-K1): track 322.2 -> 0.00 mm
- net Net-(D1-K2): track 321.5 -> 0.00 mm
- net Net-(D19-K1): track 310.2 -> 0.00 mm
- net Net-(D19-K2): track 309.3 -> 0.00 mm
- net Net-(D12-K3): track 307.3 -> 0.00 mm
- net Net-(D13-K1): track 307.1 -> 0.00 mm
- net Net-(D12-K2): track 306.3 -> 0.00 mm
- net Net-(D13-K2): track 306.1 -> 0.00 mm
- net Net-(D19-K3): track 306.1 -> 0.00 mm
- net Net-(D10-K1): track 305.3 -> 0.00 mm
- net Net-(D13-K3): track 304.0 -> 0.00 mm
- net Net-(D25-K2): track 302.7 -> 0.00 mm
- net Net-(D25-K1): track 302.1 -> 0.00 mm, vias 4 -> 0
- net Net-(D25-K3): track 299.0 -> 0.00 mm
- net Row 1: track 330.9 -> 58.5 mm, vias 2 -> 0
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- removed copper zone on B.Cu, net +3V3
- removed copper zone on F.Cu, net GND
- removed copper zone on B.Cu, net VBUS
Other:
- board outline removed

Commit message: files cleanup added edge cuts
Parts:
- C1, C10, C11, C12, C13, C14, C15, C16, C17, C2, C3, C4, C5, C6, C7, C8, C9: footprint Capacitor_SMD:C_0805_2012Metric -> Capacitor_SMD:C_0402_1005Metric
- R1, R2, R3, R4, R5, R6, R7: footprint Resistor_SMD:R_0805_2012Metric -> Resistor_SMD:R_0402_1005Metric
- moved Y1 276.7 mm to (205.5, 93.8), turned to 0 degrees
- moved C2 265.0 mm to (208.2, 93.8), turned to 90 degrees
- moved C15 264.8 mm to (202.3, 96.1), turned to 0 degrees
- moved C6 259.1 mm to (202.3, 97.1), turned to 0 degrees
- moved C1 259.1 mm to (202.3, 94.0), turned to 0 degrees
- moved C13 258.8 mm to (196.3, 89.7), turned to 90 degrees
- moved C16 258.7 mm to (196.3, 101.8), turned to -90 degrees
- moved R3 256.2 mm to (202.3, 95.0), turned to 0 degrees
- moved C9 252.3 mm to (192.7, 101.8), turned to -90 degrees
- moved C14 251.7 mm to (189.2, 95.7)
- moved C12 249.0 mm to (189.2, 94.7)
- moved C8 248.8 mm to (189.2, 97.5)
- moved C11 248.8 mm to (189.2, 99.7)
- moved C10 248.8 mm to (189.2, 98.7)
- moved R2 245.5 mm to (191.7, 87.7)
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Routing:
- net Row 1: track 58.5 -> 305.4 mm, vias 0 -> 2
- net Row 2: track 60.7 -> 275.0 mm, vias 0 -> 2
- net Row 3: track 61.0 -> 271.4 mm, vias 0 -> 2
- net GND: track 0.00 -> 199.3 mm, vias 0 -> 24
- net +3V3: track 0.00 -> 126.9 mm
- net Col 4: track 0.00 -> 48.8 mm, vias 0 -> 3
- net Col 6: track 0.00 -> 48.7 mm, vias 0 -> 3
- net Col 3: track 0.00 -> 48.6 mm, vias 0 -> 3
- net VBUS: track 0.00 -> 43.2 mm, vias 0 -> 2
- net Net-(D31-A1): track 0.00 -> 25.9 mm
- net Net-(D4-A1): track 0.00 -> 25.9 mm
- net /QSPI_SD3: track 0.00 -> 17.8 mm
- net /QSPI_SCLK: track 0.00 -> 15.5 mm
- net Net-(D4-A3): track 0.00 -> 13.8 mm
- net Net-(D31-A3): track 0.00 -> 13.8 mm
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- added copper zone on B.Cu, net +3V3
- added copper zone on F.Cu, net GND
Other:
- board outline added: 323.9 x 98.9 mm
