File: pcb_and_schematic/SKBD/SKBD.kicad_sch (KiCad schematic)
At the start: 150 parts, among them J2 USB_C_Receptacle_USB2.0_14P, SW1 ROT_SKYLOONG_HS, SW10 ROT_SKYLOONG_HS, SW11 ROT_SKYLOONG_HS, SW12 Push_Button, SW2 ROT_SKYLOONG_HS, SW3 ROT_SKYLOONG_HS, SW4 ROT_SKYLOONG_HS, SW5 ROT_SKYLOONG_HS, SW6 ROT_SKYLOONG_HS, SW7 ROT_SKYLOONG_HS, SW8 ROT_SKYLOONG_HS, SW9 ROT_SKYLOONG_HS, U2 NCP1117-3.3_SOT223, U3 W25Q128JVS, U4 RP2040, Y1 ABM8-272-T3

Commit message: revert to old desing
Parts:
- removed J2: USB_C_Receptacle_USB2.0_14P, Connector_USB:USB_C_Receptacle_JAE_DX07S016JA1R1500, symbol Connector:USB_C_Receptacle_USB2.0_14P
- added D36: PRTR5V0U2X, Package_TO_SOT_SMD:SOT-143, symbol Power_Protection:PRTR5V0U2X
- added USB1: HRO-TYPE-C-31-M-12, Type-C:HRO-TYPE-C-31-M-12-Assembly, symbol Type-C:HRO-TYPE-C-31-M-12
- C1, C10, C11, C12, C13, C14, C15, C16, C2, C5, C6, C7, C8, C9: footprint Capacitor_SMD:C_0402_1005Metric -> Capacitor_SMD:C_0805_2012Metric
- R1, R2, R3, R4, R5: footprint Resistor_SMD:R_0402_1005Metric -> Resistor_SMD:R_0805_2012Metric
- R6, R7: footprint Resistor_SMD:R_01005_0402Metric -> Resistor_SMD:R_0805_2012Metric
Connections:
- net GND: now also D36.1 (GND), USB1.1 (GND), USB1.12 (GND), USB1.13 (SHIELD)
- net Row 1: no longer D4.4 (K3), D4.5 (K2), D5.4 (K3), D5.5 (K2)
- net Row 2: now also D1.5 (K2), D2.5 (K2), D3.5 (K2), D31.5 (K2), D4.5 (K2), D5.5 (K2), D6.5 (K2), U4.3 (GPIO1)
- net Row 3: now also D1.6 (K1), D2.4 (K3), D3.4 (K3), D31.4 (K3), D4.4 (K3), D5.4 (K3), D6.4 (K3), U4.4 (GPIO2)
- net Row 4: now also D10.6 (K1), D11.6 (K1), D12.6 (K1), D32.6 (K1), D7.4 (K3), D8.6 (K1), D9.6 (K1), U4.5 (GPIO3)
- net Row 5: now also D10.5 (K2), D11.5 (K2), D12.5 (K2), D32.5 (K2), D7.5 (K2), D8.5 (K2), D9.5 (K2), U4.6 (GPIO4)
- net USB_D+: now also D36.3 (I/O2), USB1.6 (DP1), USB1.8 (DP2)
- net USB_D-: now also D36.2 (I/O1), USB1.5 (DN2), USB1.7 (DN1)
- net VBUS: now also D36.4 (VCC), USB1.11 (VBUS), USB1.2 (VBUS)
- net Col 7: now reaches MX11.1, MX23.1, MX35.1, MX47.1, MX58.1
- net Col 7: now also MX10.1, MX12.1, MX22.1, MX24.1, MX34.1, MX36.1, MX46.1, MX48.1, MX57.1, MX59.1, U4.31 (GPIO20)
- net Col 4: now reaches MX61.1, MX62.1, MX63.1, MX64.1, MX65.1, MX66.1, MX67.1, MX68.1, MX69.1, MX70.1, MX71.1, MX72.1, SW11.C
- net Col 4: now also U4.29 (GPIO18)
- net Col 2: now reaches MX1.1, MX13.1, MX14.1, MX15.1, MX2.1, MX25.1, MX26.1, MX27.1, MX3.1, MX37.1, MX38.1, MX39.1, MX49.1, MX50.1, MX51.1
- net Col 2: now also U4.27 (GPIO16)
- net Row 6: now reaches D12.4 (K3), D32.4 (K3), D7.6 (K1), D8.4 (K3), D9.4 (K3)
- net Row 6: now also D10.4 (K3), D11.4 (K3), U4.7 (GPIO5)
- net Col 6: now reaches MX19.1, MX31.1, MX43.1, MX60.1, MX7.1
- net Col 6: now also MX20.1, MX21.1, MX32.1, MX33.1, MX44.1, MX45.1, MX55.1, MX56.1, MX8.1, MX9.1, U4.30 (GPIO19)
- net at R6.1: now also USB1.4 (CC1)
- net at R7.1: now also USB1.10 (CC2)
- net Col 3: now reaches MX16.1, MX17.1, MX18.1, MX28.1, MX29.1, MX30.1, MX4.1, MX40.1, MX41.1, MX42.1, MX5.1, MX52.1, MX53.1, MX54.1, MX6.1
- net Col 3: now also U4.28 (GPIO17)
- net Row 10: now reaches D19.4 (K3), D20.6 (K1), D21.6 (K1), D22.6 (K1), D23.6 (K1), D24.6 (K1), D34.6 (K1)
- net Row 10: now also U4.12 (GPIO9); no longer D22.4 (K3), D22.5 (K2), D23.4 (K3), D23.5 (K2)
- net Row 12: now reaches D19.6 (K1), D20.4 (K3), D21.4 (K3), D24.4 (K3), D34.4 (K3)
- net Row 12: now also D22.4 (K3), D23.4 (K3), U4.14 (GPIO11)
- net Row 11: now reaches D19.5 (K2), D20.5 (K2), D21.5 (K2), D24.5 (K2), D34.5 (K2)
- net Row 11: now also D22.5 (K2), D23.5 (K2), U4.13 (GPIO10)
- net Row 9: now reaches D13.6 (K1), D14.4 (K3), D15.4 (K3), D18.4 (K3), D33.4 (K3)
- net Row 9: now also D16.4 (K3), D17.4 (K3), U4.11 (GPIO8)
- net Row 8: now reaches D13.5 (K2), D14.5 (K2), D15.5 (K2), D18.5 (K2), D33.5 (K2)
- net Row 8: now also D16.5 (K2), D17.5 (K2), U4.9 (GPIO7)
- net Row 7: now reaches D13.4 (K3), D14.6 (K1), D15.6 (K1), D16.6 (K1), D17.6 (K1), D18.6 (K1), D33.6 (K1)
- net Row 7: now also U4.8 (GPIO6); no longer D16.4 (K3), D16.5 (K2), D17.4 (K3), D17.5 (K2)
- net Col 8: now reaches SW10.C, SW2.C, SW4.C, SW6.C, SW8.C
- net Col 8: now also U4.32 (GPIO21)
- net Row 14: now reaches D25.4 (K3), D26.4 (K3), D27.4 (K3), D28.4 (K3), D29.4 (K3), D30.4 (K3), D35.4 (K3)
- net Row 14: now also U4.15 (GPIO12); no longer D28.5 (K2), D28.6 (K1), D29.5 (K2), D29.6 (K1)
- net Col 1: now reaches SW1.C, SW3.C, SW5.C, SW7.C, SW9.C
- net Col 1: now also U4.18 (GPIO15)
- net Row 15: now reaches D25.5 (K2), D26.5 (K2), D27.5 (K2), D30.5 (K2), D35.6 (K1)
- net Row 15: now also D28.5 (K2), D29.5 (K2), U4.16 (GPIO13)
- net Row 16: now reaches D25.6 (K1), D26.6 (K1), D27.6 (K1), D30.6 (K1), D35.5 (K2)
- net Row 16: now also D28.6 (K1), D29.6 (K1), U4.17 (GPIO14)
- no-connect marks 0 -> 2
Other:
- moved on the sheet: C3, C4, R6, R7, U2

Commit message: files cleanup added edge cuts
Parts:
- C1, C10, C11, C12, C13, C14, C15, C16, C17, C2, C3, C4, C5, C6, C7, C8, C9: footprint Capacitor_SMD:C_0805_2012Metric -> Capacitor_SMD:C_0402_1005Metric
- R1, R2, R3, R4, R5, R6, R7: footprint Resistor_SMD:R_0805_2012Metric -> Resistor_SMD:R_0402_1005Metric
Changed lines of the file:
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@@
 			)
 		)
-		(property "Footprint" "Capacitor_SMD:C_0805_2012Metric"
+		(property "Footprint" "Capacitor_SMD:C_0402_1005Metric"
 			(at 562.3052 107.95 0)
 			(effects
@@
 			)
 		)
-		(property "Footprint" "Resistor_SMD:R_0805_2012Metric"
+		(property "Footprint" "Resistor_SMD:R_0402_1005Metric"
 			(at 514.35 132.842 90)
 			(effects
@@
 			)
 		)
-		(property "Footprint" "Resistor_SMD:R_0805_2012Metric"
+		(property "Footprint" "Resistor_SMD:R_0402_1005Metric"
 			(at 248.92 336.042 90)
 			(effects
@@
 			)
 		)
-		(property "Footprint" "Capacitor_SMD:C_0805_2012Metric"
+		(property "Footprint" "Capacitor_SMD:C_0402_1005Metric"
 			(at 549.6052 203.2 0)
 			(effects
@@
 			)
 		)
-		(property "Footprint" "Resistor_SMD:R_0805_2012Metric"
+		(property "Footprint" "Resistor_SMD:R_0402_1005Metric"
 			(at 262.382 322.58 90)
 			(effects
@@
 			)
 		)
-		(property "Footprint" "Capacitor_SMD:C_0805_2012Metric"
+		(property "Footprint" "Capacitor_SMD:C_0402_1005Metric"
 			(at 439.1152 107.95 0)
 			(effects
@@
 			)
 		)
-		(property "Footprint" "Capacitor_SMD:C_0805_2012Metric"
+		(property "Footprint" "Capacitor_SMD:C_0402_1005Metric"
 			(at 493.7252 107.95 0)
 			(effects
@@
 			)
 		)
-		(property "Footprint" "Capacitor_SMD:C_0805_2012Metric"
+		(property "Footprint" "Capacitor_SMD:C_0402_1005Metric"
 			(at 550.8752 107.95 0)
 			(effects
@@
 			)
 		)
-		(property "Footprint" "Capacitor_SMD:C_0805_2012Metric"
+		(property "Footprint" "Capacitor_SMD:C_0402_1005Metric"
 			(at 150.8252 332.74 0)
 			(effects
@@
 			)
 		)
-		(property "Footprint" "Capacitor_SMD:C_0805_2012Metric"
+		(property "Footprint" "Capacitor_SMD:C_0402_1005Metric"
 			(at 516.5852 107.95 0)
 			(effects
@@
 			)
 		)
-		(property "Footprint" "Capacitor_SMD:C_0805_2012Metric"
+		(property "Footprint" "Capacitor_SMD:C_0402_1005Metric"
 			(at 539.4452 107.95 0)
 			(effects
@@
 			)
 		)
-		(property "Footprint" "Capacitor_SMD:C_0805_2012Metric"
+		(property "Footprint" "Capacitor_SMD:C_0402_1005Metric"
 			(at 374.65 331.1652 0)
 			(effects
@@
 			)
 		)
-		(property "Footprint" "Resistor_SMD:R_0805_2012Metric"
+		(property "Footprint" "Resistor_SMD:R_0402_1005Metric"
 			(at 514.35 140.462 90)
 			(effects
@@
 			)
 		)
-		(property "Footprint" "Capacitor_SMD:C_0805_2012Metric"
+		(property "Footprint" "Capacitor_SMD:C_0402_1005Metric"
 			(at 493.7252 123.19 0)
 			(effects
@@
 			)
 		)
-		(property "Footprint" "Resistor_SMD:R_0805_2012Metric"
+		(property "Footprint" "Resistor_SMD:R_0402_1005Metric"
 			(at 411.48 338.582 90)
 			(effects
@@
 			)
 		)
-		(property "Footprint" "Resistor_SMD:R_0805_2012Metric"
+		(property "Footprint" "Resistor_SMD:R_0402_1005Metric"
 			(at 109.474 331.216 90)
 			(effects
@@
 			)
 		)
-		(property "Footprint" "Capacitor_SMD:C_0805_2012Metric"
+		(property "Footprint" "Capacitor_SMD:C_0402_1005Metric"
 			(at 305.7652 322.58 0)
 			(effects
@@
 			)
 		)
-		(property "Footprint" "Capacitor_SMD:C_0805_2012Metric"
+		(property "Footprint" "Capacitor_SMD:C_0402_1005Metric"
 			(at 439.1152 123.19 0)
 			(effects
@@
 			)
 		)
-		(property "Footprint" "Capacitor_SMD:C_0805_2012Metric"
+		(property "Footprint" "Capacitor_SMD:C_0402_1005Metric"
 			(at 505.1552 107.95 0)
 			(effects
@@
 			)
 		)
-		(property "Footprint" "Capacitor_SMD:C_0805_2012Metric"
+		(property "Footprint" "Capacitor_SMD:C_0402_1005Metric"
 			(at 115.2652 332.74 0)
 			(effects
@@
 			)
 		)
-		(property "Footprint" "Capacitor_SMD:C_0805_2012Metric"
+		(property "Footprint" "Capacitor_SMD:C_0402_1005Metric"
 			(at 427.6852 107.95 0)
 			(effects
@@
 			)
 		)
-		(property "Footprint" "Resistor_SMD:R_0805_2012Metric"
+		(property "Footprint" "Resistor_SMD:R_0402_1005Metric"
 			(at 109.474 346.456 90)
 			(effects
@@
 			)
 		)
-		(property "Footprint" "Capacitor_SMD:C_0805_2012Metric"
+		(property "Footprint" "Capacitor_SMD:C_0402_1005Metric"
 			(at 374.65 341.3252 0)
 			(effects
@@
 			)
 		)
-		(property "Footprint" "Capacitor_SMD:C_0805_2012Metric"
+		(property "Footprint" "Capacitor_SMD:C_0402_1005Metric"
 			(at 528.0152 107.95 0)
 			(effects
